File: hardware/dev-bench/cad/plytka-nosna.kicad_sch (KiCad schematic)
At the start: 59 parts, among them J1 ARDUINO POWER, J10 CC1120EM P2, J11 ANALIZATOR, J12 VTEST 0-15V, J2 ARDUINO A0-A5, J3 ARDUINO D0-D7, J4 ARDUINO D8-SCL, J5 DEVKITC J1, J6 DEVKITC J3, J7 SHARP 4694, J8 FRAM 4719, J9 CC1120EM P1, Q1 MMBT3904, SW1 GÓRA, SW2 DÓŁ, SW3 OK, SW4 WSTECZ, SW5 CISZA, SW6 PRZYGOTOWANIE

Commit message: Dev bench: carrier N1 after review, fabrication files for a test build
Review of N1 (electrical, mechanical, docs) found no critical defect;
fixes applied in the generators:
- buzzer from +5V through 22 ohm 1206, not from the radio's 3.0 V rail
- 1k in series with the CISZA switch, 33 ohm series on SCK at both MCUs,
  2k2 pull-down on LCD_DISP, BAT54S clamp on VTEST, RF_RESET pull-down 10k
- JP3 feeds the CC1120EM (radio current measurement in bench A)
- RF_GPIO2 on ESP32 GPIO4 instead of GPIO47 (N16R16V modules fit)
- no copper on B.Cu and no vias over the DK P20 pin row, no tracks under
  standoffs and screw heads, wider P5 notch
- module outlines, SMA circle and USB mark on the silkscreen, text >=1 mm,
  J12 polarity, missing_courtyard check enabled, hole/via minima 0.4/0.8 mm
- BOM: one Adafruit 85 kit, per-part notes, shunts, caps, standoffs

ERC 0, DRC 0, 0 unconnected, 0 schematic parity. Reproduction checked with
tools/compare_boards.py (checks/odtworzenie.md). Fabrication package in
fabrication/N1, schematic PDF, assembly and bring-up procedure, list of
conditions before an order. Docs: F81 updated, R02 no longer called the
first printed board, dev-bench README on wires vs carrier.
Parts:
- added D3: BAT54S, Package_TO_SOT_SMD:SOT-23, symbol Diode:BAT54S
- added JP3: 3V3 RADIO A, Connector_PinHeader_2.54mm:PinHeader_1x02_P2.54mm_Vertical, symbol Connector_Generic:Conn_01x02
- added R16: 1k, Resistor_SMD:R_0805_2012Metric, symbol Device:R
- added R17, R18: 33R, Resistor_SMD:R_0805_2012Metric, symbol Device:R
- added R19: 2k2, Resistor_SMD:R_0805_2012Metric, symbol Device:R
- R12: value 100k -> 10k; MPN RC0805FR-07100KL -> RC0805FR-0710KL
- R2: value 10R -> 22R; footprint Resistor_SMD:R_0805_2012Metric -> Resistor_SMD:R_1206_3216Metric; MPN RC0805FR-0710RL -> RC1206FR-0722RL
Connections:
- net +3V3: now also D3.2 (K), JP3.1 (Pin_1); no longer C1.1, C2.1, J10.7 (Pin_7), J10.9 (Pin_9), R2.1
- net +5V: now also R2.1
- net GND: now also D3.1 (A), R19.2
- net LCD_DISP: now also R19.1
- net RF_GPIO2: now also J5.4 (Pin_4); no longer J6.17 (Pin_17)
- net SPI_SCK: now also R17.2, R18.2; no longer J3.4 (Pin_4), J5.18 (Pin_18)
- net SW_CISZA: now also R16.2; no longer SW5.2 (B)
- net VTEST: now also D3.3 (COM)
- new net +3V3_RF: C1.1, C2.1, J10.7 (Pin_7), J10.9 (Pin_9), JP3.2 (Pin_2)
- new net SPI_SCK_DEVKIT: J5.18 (Pin_18), R18.1
- new net SPI_SCK_DK: J3.4 (Pin_4), R17.1
- new net SW_COM: R16.1, SW5.2 (B)
Other:
- moved on the sheet: C1, C2, C3, C5, J11, J12, J8, R11, R12, R14, R15
