File: hardware/przetwornica-3v3/cad/przetwornica-3v3.kicad_pcb (KiCad board)
At the start: 4 copper layers, 56 x 48 mm, 39 parts, among them J1 VIN, J2 VOUT, U1 LTC3115EFE-1#PBF

Commit message: Płytka przetwornicy: biegunowość zacisków, powtarzalny eksport, CPL listew
Przy J1 i J2 nie było oznaczenia biegunowości, a płytka nie ma ochrony
przed odwrotnym podłączeniem. Sitodruk dostaje znaki „+” i „−” przy
końcach zacisków (korpusy zasłaniają pady): J1 ma GND u góry i VIN na
dole, J2 VOUT u góry i GND na dole. README opisuje biegunowość i
zaleca pierwsze włączenie z ograniczeniem prądu.

Strefy VIN i VOUT dostają priorytet 4, wyższy niż węzły przełączające.
Przy równym priorytecie kolejność wypełniania decydowała, która strefa
zachowuje pasek odstępu (około 0,19 mm²), więc kolejne eksporty dawały
różną miedź. Teraz dwa eksporty dają identyczne Gerbery.

JLC ma modele listew obrócone o 90° względem KiCad (podgląd z
2026-10-31), więc CPL obraca JP1–JP5 tak jak U1.

Co-Authored-By: Claude Opus 5.5 <noreply@anthropic.com>
Signed-off-by: Tomek Mierzwa <16899265+tmierzwa@users.noreply.github.com>
Other:
- board text added: "+"
- board text added: "−"
